Commit message: zeros adjusted

File: silverhand_arm_description/urdf/silverhand.urdf (robot description, URDF)
Before this commit: robot silverhand, 7 links, 6 joints
Joints:
- joint joint_1: origin xyz=0 0 0.003445 rpy=3.1416 -1.0248E-21 -1.6736E-05 -> xyz=0 0 0.003445 rpy=3.1416 0 0
- joint joint_2: origin xyz=0 0.064146 -0.16608 rpy=1.5708 0.5236 -1.5708 -> xyz=0 0.064146 -0.16608 rpy=1.5708 0 -1.5708
- joint joint_3: origin xyz=0.1525 -0.26414 0 rpy=3.3431E-16 -1.4164E-16 -1.4953816339 -> xyz=0.1525 -0.26414 0 rpy=0 0 0

File: silverhand_arm_description/urdf/silverhand.urdf.xacro (robot description, xacro)
@@ -1,4 +1,5 @@
 <?xml version="1.0"?>
 <robot xmlns:xacro="http://www.ros.org/wiki/xacro" name="silverhand">
+  <xacro:include filename="$(find silverhand_arm_description)/urdf/silverhand_macro.urdf.xacro"/>
   <xacro:arg
     name="initial_positions_file"
@@ -7,6 +8,6 @@
   <xacro:arg name="can_iface" default="can0"/>
   <xacro:arg name="node_id" default="100"/>
-  <xacro:include filename="$(find silverhand_arm_description)/urdf/silverhand.urdf"/>
   <xacro:include filename="$(find silverhand_arm_description)/ros2_control/silverhand.ros2_control.xacro"/>
+  <xacro:silverhand_arm prefix=""/>
   <xacro:silverhand_ros2_control
     name="SilverhandArmSystem"
